File: PTPseminarLNv2/PTPseminarLNv2.kicad_sch (KiCad schematic)
At the start: 39 parts, among them J1 SIM2, J5 CORTEX SWD, J6 USB_B_Micro, SW1 SW_SPDT, SW2 SW_DPST_x2, U1 SIM808, U2 STM32F103C8Tx, U3 SSD1306, U4 LM1117DT-3.3

Commit message: skoro gotovi
na najjace
Parts:
- AE1, AE2: Availability In Stock -> (none); Check_prices https://www.snapeda.com/parts/7488910915/W%25C3%25BCrth+Ele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 -> (none); Description_1 RF ANTENNA Bluetooth, GPS, GSM, LTE, Wi-Fi, WLAN, Zigbee™ C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 -> (none); MF Würth Elektronik -> (none); MP 7488910915 -> (none); Manufacturer (none) -> Würth Elektronik; Manufacturer part number (none) -> 7488910915; Package None -> (none); Price None -> (none); SnapEDA_Link https://www.snapeda.com/parts/7488910915/W%25C3%25BCrth+Ele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 -> (none)
- C1, C3, C7: Manufacturer (none) -> Murata Manufacturing Co.; Manufacturer part number (none) -> GRM31CR71H104KA88L
- C10, C11, C8: Manufacturer (none) -> Murata Manufacturing Co.; Manufacturer part number (none) -> GRM31CR61C106KA12L
- C2: Manufactuer (none) -> Murata Manufacturing Co.; Manufactuer part number (none) -> GRM31CR71H104KA88L
- C4: value 10uF -> 10u; Manufacturer  (none) -> Murata Manufacturing Co.; Manufacturer part number (none) -> GRM31CR61C106KA12L
- C5: value 10uF -> 10u; Manufacturer (none) -> Murata Manufacturing Co.; Manufacturer part number (none) -> GRM31CR61C106KA12L
- C6: Manufacturer  (none) -> Murata Manufacturing Co.; Manufacturer part number (none) -> GRM31CR71H104KA88L
- C9: Manufacturer (none) -> Murata Manufacturing Co.; Manufacturer part number (none) -> GRM31CR71H103KA01L
- D1, D2: Manufacturer (none) -> Lite-On; Manufacturer part number (none) -> LTST-C191KRKT
- FB1: Manufacturer (none) -> Murata Manufacturing Co.; Manufacturer part number (none) -> BLM31AG121SN1L
- J1: Manufacturer (none) -> TE Connectivity; Manufacturer part number (none) -> 2452808-1
- J2: Manufacturer (none) -> JST; Manufacturer part number (none) -> B2B-XH-A
- J3, J4: Manufacturer (none) -> JST; Manufacturer part number (none) -> B4B-PH-K-S
- J5: Manufacturer (none) -> Tag-Connect; Manufacturer part number (none) -> TC2030-CTX
- J6: Manufacturer (none) -> Belden Inc.; Manufacturer part number (none) -> 2486 01
- R1, R2: Manufacturer (none) -> Yageo Corporation; Manufacturer part number (none) -> RC1206JR-07100KL
- R3, R4, R5: Manufacturer (none) -> Yageo Corporation; Manufacturer part number (none) -> RC1206JR-0722RL
- R6: Manufacturer (none) -> Yageo Corporation; Manufacturer part number (none) -> RC1206JR-0710KL
- R7: Manufacturer (none) -> Yageo Corporation; Manufacturer part number (none) -> RC1206JR-071K5L
- SW1: Manufacturer (none) -> C&K Components (Littelfuse); Manufacturer part number (none) -> OS102011MS2Q
- SW2: Manufacturer (none) -> Omron Electronics; Manufacturer part number (none) -> A6S-1101
- U1: Availability In Stock -> (none); Check_prices https://www.snapeda.com/parts/SIM808/SIMCom/view-part/?ref=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 -> (none); Description_1 SIM808 GPS, GPRS/GSM RF mikroBUS™ Click™ Platform Evaluatio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 -> (none); MANUFACTURER SIMCOM -> (none); MAXIMUM_PACKAGE_HEIGHT 2.8mm -> (none); MF SIMcom Wireless solutions Co.,Ltd -> (none); MP SIM808 -> (none); Manufacturer (none) -> SIMcom Wireless solutions Co.,Ltd; Manufacturer part number (none) -> XCVR_SIM808; PARTREV 1.03 -> (none); Package None -> (none); Price None -> (none); STANDARD Manufacturer recommendations -> (none); SnapEDA_Link https://www.snapeda.com/parts/SIM808/SIMCom/view-part/?ref=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 -> (none)
- U2: Manufacturer (none) -> STMicroelectronics; Manufacturer part number (none) -> STM32F103C8Tx
- U3: Availability Not in stock -> (none); Check_prices https://www.snapeda.com/parts/DM-OLED096-636/Display+Module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 -> (none); Description_1 0.96” 128 X 64 MONOCHROME GRAPHIC OLED DISPLAY MODULE - I2C -> (none); MANUFACTURER Displaymodule -> (none); MAXIMUM_PACKAGE_HEIGHT 11.3 mm -> (none); MF Display Module -> (none); MP DM-OLED096-636 -> (none); Manufacturer (none) -> Display Module; Manufacturer part number (none) -> DM-OLED096-636; PARTREV 2018-09-10 -> (none); Package Package -> (none); Price None -> (none); STANDARD Manufacturer Recommendations -> (none); SnapEDA_Link https://www.snapeda.com/parts/DM-OLED096-636/Display+Module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 -> (none)
- U4: Manufacturer (none) -> Texas Instruments; Manufacturer part number (none) -> LM1117DT-3.3/NOPB
Other:
- note added: "Antene"
- note added: "GPS i GSM"
- note added: "Indikatori"
- note added: "Konektori"
- note added: "Mounting holes"
- note added: "Napajanje"
- note added: "OLED screen"
- note added: "ON/OFF Switch"
- note added: "SIM kartica"
- note added: "STM Mikroupravljač"
- note added: "Ulazi za komunikaciju"
- moved on the sheet: C4, C5, D1, D2, H1, H2, H3, H4, J5, J6, R1, R2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
