File: PTPseminarLNv2/PTPseminarLNv2.kicad_pcb (KiCad board)
At the start: 2 copper layers, 91 x 79 mm, 39 parts, among them J1 SIM2, J5 CORTEX SWD, J6 USB_B_Micro, SW1 SW_SPDT, SW2 SW_DPST_x2, U1 SIM808, U2 STM32F103C8Tx, U3 SSD1306, U4 LM1117DT-3.3

Commit message: bato
naanajjace
Parts:
- moved AE1 71.5 mm to (158.0, 129.0), turned to 180 degrees
- moved FB1 5.06 mm to (173.0, 78.5), turned to 180 degrees
- moved J5 4.47 mm to (171.3, 127.7)
Routing:
- net GND: track 0.00 -> 372.3 mm, vias 0 -> 23
- net +3.3V: track 44.8 -> 317.2 mm, vias 0 -> 5
- net VD: track 43.9 -> 129.3 mm, vias 0 -> 4
- net POWERSW: track 21.8 -> 105.9 mm, vias 2 -> 6
- net SWCLK: track 0.00 -> 55.3 mm, vias 0 -> 2
- net SWDIO: track 0.00 -> 53.0 mm, vias 0 -> 2
- net Net-(D2-A): track 0.00 -> 51.7 mm
- net Net-(D1-A): track 0.00 -> 49.8 mm
- net RX: track 29.9 -> 79.7 mm, vias 0 -> 4
- net GPSANT: track 0.00 -> 36.4 mm
- net /SW_BOOT0: track 0.00 -> 34.5 mm, vias 0 -> 2
- net USB_D+: track 9.81 -> 42.8 mm, vias 0 -> 2
- net +3.3VA: track 0.00 -> 28.2 mm
- net SDA: track 17.8 -> 37.7 mm, vias 0 -> 2
- net /BOOT0: track 0.00 -> 18.1 mm
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- added copper zone on B.Cu, net GND
Other:
- outline, holes or cut-outs redrawn

Commit message: skoro gotovi
na najjace
Routing:
- net TX: track 69.7 -> 71.7 mm

Commit message: uf
oke
Routing:
- net VD: track 129.3 -> 128.8 mm
Changed lines of the file:
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@@
 		(at 171.254 127.746 90)
 		(property "Reference" "J5"
-			(at 5.246 -7.254 180)
+			(at 5.496 -7.254 180)
 			(layer "F.SilkS")
 			(effects
 				(font
-					(size 0.48 0.48)
-					(thickness 0.12)
+					(size 1 1)
+					(thickness 0.15)
 				)
 			)
@@
 		(tags "capacitor handsolder")
 		(property "Reference" "C10"
-			(at 0 -1.65 90)
+			(at -3.4375 -0.15 180)
 			(layer "F.SilkS")
 			(effects
@@
 		(tags "capacitor handsolder")
 		(property "Reference" "C11"
-			(at 0 -1.75 90)
+			(at -3.4375 -0.25 180)
 			(layer "F.SilkS")
 			(effects
@@
 		(tags "capacitor handsolder")
 		(property "Reference" "C2"
-			(at 0 -1.55 90)
+			(at 3.1875 -0.05 180)
 			(layer "F.SilkS")
 			(effects
@@
 		(tags "capacitor handsolder")
 		(property "Reference" "C9"
-			(at 0 -1.55 90)
+			(at -3.4375 -0.05 180)
 			(layer "F.SilkS")
 			(effects
@@
 		(tags "resistor handsolder")
 		(property "Reference" "R1"
-			(at 0 -1.83 90)
+			(at -3.45 0 180)
 			(layer "F.SilkS")
 			(effects
@@
 		(tags "capacitor handsolder")
 		(property "Reference" "C6"
-			(at 0 -1.65 90)
+			(at 3.1875 -0.15 180)
 			(layer "F.SilkS")
 			(effects
@@
 		(tags "resistor handsolder")
 		(property "Reference" "R2"
-			(at 0 -1.83 90)
+			(at -3.45 0 180)
 			(layer "F.SilkS")
 			(effects
@@
 		(tags "capacitor handsolder")
 		(property "Reference" "C7"
-			(at 0 -1.5 90)
+			(at 3.1875 -0.5 180)
 			(layer "F.SilkS")
 			(effects
@@
 	)
 	(segment
-		(start 102 106.75)
-		(end 102 107)
-		(width 0.5)
-		(layer "F.Cu")
-		(net 5)
-	)
-	(segment
 		(start 173.75 132)
 		(end 170 132)
@@
 	)
 	(segment
-		(start 111.5 72.5)
-		(end 112 72.5)
-		(width 0.5)
-		(layer "F.Cu")
-		(net 6)
-	)
-	(segment
 		(start 121.10766 64.984603)
 		(end 118.515397 64.984603)
@@
 	)
 	(segment
-		(start 125.5 103.5)
-		(end 125.625 103.375)
-		(width 0.5)
-		(layer "B.Cu")
-		(net 18)
-	)
-	(segment
-		(start 128 101)
-		(end 128.5 100.5)
-		(width 0.5)
-		(layer "B.Cu")
-		(net 18)
-	)
-	(segment
-		(start 125.625 103.375)
+		(start 128.5 100.5)
 		(end 124.5 104.5)
 		(width 0.5)
@@
 		(width 0.5)
 		(layer "B.Cu")
-		(net 18)
-	)
-	(segment
-		(start 125.625 103.375)
-		(end 128 101)
-		(width 0.5)
-		(layer "B.Cu")

Commit message: finito
fin
Routing:
- added copper zone on F.Cu, net GND
Changed lines of the file:
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@@
+		(net 3)
+		(net_name "GND")
+		(layer "F.Cu")
+		(hatch edge 0.5)
+		(priority 2)
+		(connect_pads
+			(clearance 0.5)
+		)
+		(min_thickness 0.25)
+		(filled_areas_thickness no)
+		(fill yes
+			(thermal_gap 0.5)
+			(thermal_bridge_width 0.5)
+		)
+		(polygon
+			(pts
+				(xy 156.75 59.25) (xy 163.25 59.25) (xy 163.25 56.5) (xy 156.75 56.5)
+			)
+		)
+	)
+	(zone
+		(net 3)
+		(net_name "GND")
+		(layer "F.Cu")
+		(hatch edge 0.5)
+		(priority 1)
+		(connect_pads
+			(clearance 0.5)
+		)
+		(min_thickness 0.25)
+		(filled_areas_thickness no)
+		(fill yes
+			(thermal_gap 0.5)
+			(thermal_bridge_width 0.5)
+		)
+		(polygon
+			(pts
+				(xy 155 128.25) (xy 161.25 128.25) (xy 161.25 131) (xy 155 131)
+			)
+		)
+	)
+	(zone
 		(net 3)
 		(net_name "GND")
